Commit message: works?

File: src/xarm_description/urdf/lite6/lite6.urdf.xacro (robot description, xacro)
@@ -13,8 +13,8 @@
     <xacro:property name="default_inertial_params_filename" value="xarm6_type9_HT_BR2"/>
     <xacro:if value="${inertial_params_filename != ''}">
-      <xacro:property name="link_inertial_params_file" value="$(find xarm_description)/config/link_inertial/${inertial_params_filename}.yaml"/>
+      <xacro:property name="link_inertial_params_file" value="$(arg xarm_description)/config/link_inertial/${inertial_params_filename}.yaml"/>
     </xacro:if>
     <xacro:unless value="${inertial_params_filename != ''}">
-      <xacro:property name="link_inertial_params_file" value="$(find xarm_description)/config/link_inertial/${default_inertial_params_filename}.yaml"/>
+      <xacro:property name="link_inertial_params_file" value="$(arg xarm_description)/config/link_inertial/${default_inertial_params_filename}.yaml"/>
     </xacro:unless>
     <xacro:if value="${use_xacro_load_yaml}">

File: src/xarm_description/urdf/lite6/lite6_robot_macro.xacro (robot description, xacro)
@@ -17,9 +17,9 @@
     <!-- include lite6 relative macros: -->
     <xacro:if value="${is_ros2}">
-      <xacro:include filename="$(find xarm_description)/urdf/lite6/lite6.ros2_control.xacro" />
+      <xacro:include filename="$(arg xarm_description)/urdf/lite6/lite6.ros2_control.xacro" />
     </xacro:if>
-    <xacro:include filename="$(find xarm_description)/urdf/lite6/lite6.urdf.xacro" />
-    <xacro:include filename="$(find xarm_description)/urdf/lite6/lite6.transmission.xacro" />
-    <xacro:include filename="$(find xarm_description)/urdf/lite6/lite6.gazebo.xacro" />
+    <xacro:include filename="$(arg xarm_description)/urdf/lite6/lite6.urdf.xacro" />
+    <xacro:include filename="$(arg xarm_description)/urdf/lite6/lite6.transmission.xacro" />
+    <xacro:include filename="$(arg xarm_description)/urdf/lite6/lite6.gazebo.xacro" />
     <xacro:if value="${limited}">
       <xacro:if value="${is_ros2}">

File: src/xarm_description/urdf/xarm_device.urdf.xacro (robot description, xacro)
@@ -15,5 +15,9 @@
   <xacro:arg name="report_type" default="normal"/>
   <xacro:arg name="ros2_control_plugin" default="uf_robot_hardware/UFRobotSystemHardware"/>
+  <!--
   <xacro:arg name="ros2_control_params" default="$(find xarm_controller)/config/xarm$(arg dof)_controllers.yaml"/>
+  -->
+  <xacro:arg name="ros2_control_params" default="/home/shrenikm/Projects/manipulation_research/src/xarm_controller/config/xarm$(arg dof)_controllers.yaml"/>
+  <xacro:arg name="xarm_description" default="/home/shrenikm/Projects/manipulation_research/src/xarm_description"/>
   <xacro:arg name="add_realsense_d435i" default="false"/>
   <xacro:arg name="add_d435i_links" default="true"/>
@@ -37,5 +41,8 @@
   <xacro:arg name="attach_rpy" default="0 0 0"/>
   <!-- load xarm device -->
+  <!--
   <xacro:include filename="$(find xarm_description)/urdf/xarm_device_macro.xacro" />
+  -->
+  <xacro:include filename="$(arg xarm_description)/urdf/xarm_device_macro.xacro" />
   <xacro:xarm_device prefix="$(arg prefix)" hw_ns="$(arg hw_ns)" limited="$(arg limited)"
     effort_control="$(arg effort_control)" velocity_control="$(arg velocity_control)"

File: src/xarm_description/urdf/xarm_device_macro.xacro (robot description, xacro)
@@ -40,13 +40,13 @@
     >
     <!-- Load Common Material -->
-    <xacro:include filename="$(find xarm_description)/urdf/_private_macro.xacro" />
+    <xacro:include filename="$(arg xarm_description)/urdf/_private_macro.xacro" />
     <xacro:device_macro_begin />
     <!-- Load Common Material -->
-    <xacro:include filename="$(find xarm_description)/urdf/common/common.material.xacro" />
+    <xacro:include filename="$(arg xarm_description)/urdf/common/common.material.xacro" />
     <xacro:common_material prefix="${prefix}"/>
     <!-- Specify Mesh file path -->
     <xacro:if value="${ros2_control_plugin == 'gazebo_ros2_control/GazeboSystem'}">
       <!-- gazebo use -->
-      <xacro:property name="mesh_path" value="file://$(find xarm_description)/meshes" scope="parent"/>
+      <xacro:property name="mesh_path" value="file://$(arg xarm_description)/meshes" scope="parent"/>
     </xacro:if>
     <xacro:unless value="${ros2_control_plugin == 'gazebo_ros2_control/GazeboSystem'}">
@@ -54,5 +54,5 @@
     </xacro:unless>
     <!-- include common.link.xacro -->
-    <xacro:include filename="$(find xarm_description)/urdf/common/common.link.xacro" />
+    <xacro:include filename="$(arg xarm_description)/urdf/common/common.link.xacro" />
     <xacro:parse_link_inertial_filename dof="${dof}" robot_type="${robot_type}" robot_sn="${robot_sn}" model1300="${model1300}" />
     <xacro:property name="inertial_params_filename" value="${scope_parent_inertial_params_filename}"/>
@@ -69,5 +69,5 @@
     <xacro:if value="${dof == 5}">
       <!-- Load XArm5 Robot Model URDF -->
-      <xacro:include filename="$(find xarm_description)/urdf/xarm5/xarm5_robot_macro.xacro" />
+      <xacro:include filename="$(arg xarm_description)/urdf/xarm5/xarm5_robot_macro.xacro" />
       <xacro:xarm5_robot prefix="${prefix}" hw_ns="${hw_ns}" limited="${limited}"
         effort_control="${effort_control}" velocity_control="${velocity_control}"
@@ -84,5 +84,5 @@
       <xacro:if value="${robot_type == 'lite'}">
         <!-- Load Lite6 Robot Model URDF -->
-        <xacro:include filename="$(find xarm_description)/urdf/lite6/lite6_robot_macro.xacro" />
+        <xacro:include filename="$(arg xarm_description)/urdf/lite6/lite6_robot_macro.xacro" />
         <xacro:lite6_robot prefix="${prefix}" hw_ns="${hw_ns}" limited="${limited}"
           effort_control="${effort_control}" velocity_control="${velocity_control}"
@@ -97,5 +97,5 @@
       <xacro:unless value="${robot_type == 'lite'}">
         <!-- Load XArm6 Robot Model URDF -->
-        <xacro:include filename="$(find xarm_description)/urdf/xarm6/xarm6_robot_macro.xacro" />
+        <xacro:include filename="$(arg xarm_description)/urdf/xarm6/xarm6_robot_macro.xacro" />
         <xacro:xarm6_robot prefix="${prefix}" hw_ns="${hw_ns}" limited="${limited}"
           effort_control="${effort_control}" velocity_control="${velocity_control}"
@@ -112,5 +112,5 @@
     <xacro:unless value="${dof == 5 or dof == 6}">
       <!-- Load XArm7 Robot Model URDF -->
-      <xacro:include filename="$(find xarm_description)/urdf/xarm7/xarm7_robot_macro.xacro" />
+      <xacro:include filename="$(arg xarm_description)/urdf/xarm7/xarm7_robot_macro.xacro" />
       <xacro:xarm7_robot prefix="${prefix}" hw_ns="${hw_ns}" limited="${limited}"
         effort_control="${effort_control}" velocity_control="${velocity_control}"
@@ -126,8 +126,8 @@
     <xacro:if value="${add_realsense_d435i}">
       <!-- (xarm) Load RealSense D435i URDF -->
-      <xacro:include filename="$(find xarm_description)/urdf/camera/realsense_d435i.urdf.xacro" />
+      <xacro:include filename="$(arg xarm_description)/urdf/camera/realsense_d435i.urdf.xacro" />
       <xacro:d435i_urdf prefix="${prefix}" add_d435i_links="${add_d435i_links}" />
       <xacro:if value="${add_d435i_links}">
-        <xacro:include filename="$(find xarm_description)/urdf/camera/realsense.gazebo.xacro" />
+        <xacro:include filename="$(arg xarm_description)/urdf/camera/realsense.gazebo.xacro" />
         <xacro:realsense_gazebo prefix="${prefix}" />
       </xacro:if>
@@ -144,10 +144,10 @@
       <xacro:if value="${robot_type == 'lite'}">
         <!-- Load Lite Gripper Model URDF -->
-        <xacro:include filename="$(find xarm_description)/urdf/gripper/lite_gripper.urdf.xacro" />
+        <xacro:include filename="$(arg xarm_description)/urdf/gripper/lite_gripper.urdf.xacro" />
         <xacro:uflite_gripper_urdf prefix="${prefix}" attach_to="${prefix}link_eef" />
       </xacro:if>
       <xacro:unless value="${robot_type == 'lite'}">
         <!-- Load XArm Gripper Model URDF -->
-        <xacro:include filename="$(find xarm_description)/urdf/gripper/xarm_gripper_macro.xacro" />
+        <xacro:include filename="$(arg xarm_description)/urdf/gripper/xarm_gripper_macro.xacro" />
         <xacro:xarm_gripper_macro prefix="${prefix}" attach_to="${prefix}link_eef" effort_control="${effort_control}" velocity_control="${velocity_control}"
           ros2_control_plugin="${ros2_control_plugin}" dof="${dof}" />
@@ -157,10 +157,10 @@
       <xacro:if value="${robot_type == 'lite'}">
         <!-- Load Lite Vacuum Gripper Model URDF -->
-        <xacro:include filename="$(find xarm_description)/urdf/vacuum_gripper/lite_vacuum_gripper.urdf.xacro" />
+        <xacro:include filename="$(arg xarm_description)/urdf/vacuum_gripper/lite_vacuum_gripper.urdf.xacro" />
         <xacro:uflite_vacuum_gripper_urdf prefix="${prefix}" attach_to="${prefix}link_eef" />
       </xacro:if>
       <xacro:unless value="${robot_type == 'lite'}">
         <!-- Load XArm Vacuum Gripper Model URDF -->
-        <xacro:include filename="$(find xarm_description)/urdf/vacuum_gripper/xarm_vacuum_gripper.urdf.xacro" />
+        <xacro:include filename="$(arg xarm_description)/urdf/vacuum_gripper/xarm_vacuum_gripper.urdf.xacro" />
         <xacro:xarm_vacuum_gripper_urdf prefix="${prefix}" attach_to="${prefix}link_eef" effort_control="${effort_control}" velocity_control="${velocity_control}" />
       </xacro:unless>
@@ -168,5 +168,5 @@
     <xacro:if value="${not add_gripper and not add_vacuum_gripper and add_other_geometry}">
       <!-- Load Other Model URDF -->
-      <xacro:include filename="$(find xarm_description)/urdf/other/other_geometry.urdf.xacro" />
+      <xacro:include filename="$(arg xarm_description)/urdf/other/other_geometry.urdf.xacro" />
       <xacro:other_geometry prefix="${prefix}" attach_to="${prefix}link_eef"
         geometry_type="${geometry_type}" geometry_mass="${geometry_mass}"
@@ -180,5 +180,5 @@
     <!-- gazebo_plugin -->
     <xacro:if value="${load_gazebo_plugin}">
-      <xacro:include filename="$(find xarm_description)/urdf/common/common.gazebo.xacro" />
+      <xacro:include filename="$(arg xarm_description)/urdf/common/common.gazebo.xacro" />
       <xacro:if value="${is_ros2}">
         <xacro:gazebo_ros2_control_plugin ros2_control_params="${ros2_control_params}"/>
@@ -189,5 +189,5 @@
     </xacro:if>
     <xacro:if value="${use_gazebo_camera}">
-      <xacro:include filename="$(find xarm_description)/urdf/camera/camera.gazebo.xacro" />
+      <xacro:include filename="$(arg xarm_description)/urdf/camera/camera.gazebo.xacro" />
       <xacro:camera_gazebo prefix="${prefix}" />
     </xacro:if>
