Commit message: wew works

File: src/xarm_description/urdf/gripper/lite_gripper.urdf.xacro (robot description, xacro)
@@ -18,10 +18,10 @@
       </inertial>
       <xacro:common_link_visual
-        mesh_filename="gripper/lite/visual/gripper_lite.stl"
+        mesh_filename="gripper/lite/visual/gripper_lite.obj"
         origin_xyz="0 0 0"
         origin_rpy="0 0 0"
         material_name="${prefix}White" />
       <xacro:common_link_collision
-        mesh_filename="gripper/lite/collision/gripper_lite.stl"
+        mesh_filename="gripper/lite/collision/gripper_lite.obj"
         origin_xyz="0 0 0"
         origin_rpy="0 0 0" />

File: src/xarm_description/urdf/lite6.urdf (robot description, URDF)
Before this commit: robot lite6, 9 links, 8 joints
Links:
- link link1: geometry collision mesh filename=/home/shrenikm/Projects/manipulation_research/src/xarm_desc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; visual mesh filename=/home/shrenikm/Projects/manipulation_research/src/xarm_desc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
- link link2: geometry collision mesh filename=/home/shrenikm/Projects/manipulation_research/src/xarm_desc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; visual mesh filename=/home/shrenikm/Projects/manipulation_research/src/xarm_desc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
- link link3: geometry collision mesh filename=/home/shrenikm/Projects/manipulation_research/src/xarm_desc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; visual mesh filename=/home/shrenikm/Projects/manipulation_research/src/xarm_desc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
- link link4: geometry collision mesh filename=/home/shrenikm/Projects/manipulation_research/src/xarm_desc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; visual mesh filename=/home/shrenikm/Projects/manipulation_research/src/xarm_desc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
- link link5: geometry collision mesh filename=/home/shrenikm/Projects/manipulation_research/src/xarm_desc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; visual mesh filename=/home/shrenikm/Projects/manipulation_research/src/xarm_desc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
- link link6: geometry collision mesh filename=/home/shrenikm/Projects/manipulation_research/src/xarm_desc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; visual mesh filename=/home/shrenikm/Projects/manipulation_research/src/xarm_desc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
- link link_base: geometry collision mesh filename=/home/shrenikm/Projects/manipulation_research/src/xarm_desc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; visual mesh filename=/home/shrenikm/Projects/manipulation_research/src/xarm_desc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

File: src/xarm_description/urdf/lite6/lite6.urdf.xacro (robot description, xacro)
@@ -33,10 +33,10 @@
       </inertial>
       <xacro:common_link_visual
-        mesh_filename="lite6/visual/base.stl"
-        origin_xyz="0 0 0"
-        origin_rpy="0 0 0"
-        material_name="${prefix}White" />
-      <xacro:common_link_collision
-        mesh_filename="lite6/visual/base.stl"
+        mesh_filename="lite6/visual/base.obj"
+        origin_xyz="0 0 0"
+        origin_rpy="0 0 0"
+        material_name="${prefix}White" />
+      <xacro:common_link_collision
+        mesh_filename="lite6/visual/base.obj"
         origin_xyz="0 0 0"
         origin_rpy="0 0 0" />
@@ -47,10 +47,10 @@
         origin_rpy="0 0 0"/>
       <xacro:common_link_visual
-        mesh_filename="lite6/visual/link1.stl"
-        origin_xyz="0 0 0"
-        origin_rpy="0 0 0"
-        material_name="${prefix}White" />
-      <xacro:common_link_collision
-        mesh_filename="lite6/visual/link1.stl"
+        mesh_filename="lite6/visual/link1.obj"
+        origin_xyz="0 0 0"
+        origin_rpy="0 0 0"
+        material_name="${prefix}White" />
+      <xacro:common_link_collision
+        mesh_filename="lite6/visual/link1.obj"
         origin_xyz="0 0 0"
         origin_rpy="0 0 0" />
@@ -73,10 +73,10 @@
         origin_rpy="0 0 0"/>
       <xacro:common_link_visual
-        mesh_filename="lite6/visual/link2.stl"
-        origin_xyz="0 0 0"
-        origin_rpy="0 0 0"
-        material_name="${prefix}White" />
-      <xacro:common_link_collision
-        mesh_filename="lite6/visual/link2.stl"
+        mesh_filename="lite6/visual/link2.obj"
+        origin_xyz="0 0 0"
+        origin_rpy="0 0 0"
+        material_name="${prefix}White" />
+      <xacro:common_link_collision
+        mesh_filename="lite6/visual/link2.obj"
         origin_xyz="0 0 0"
         origin_rpy="0 0 0" />
@@ -99,10 +99,10 @@
         origin_rpy="0 0 0"/>
       <xacro:common_link_visual
-        mesh_filename="lite6/visual/link3.stl"
-        origin_xyz="0 0 0"
-        origin_rpy="0 0 0"
-        material_name="${prefix}White" />
-      <xacro:common_link_collision
-        mesh_filename="lite6/visual/link3.stl"
+        mesh_filename="lite6/visual/link3.obj"
+        origin_xyz="0 0 0"
+        origin_rpy="0 0 0"
+        material_name="${prefix}White" />
+      <xacro:common_link_collision
+        mesh_filename="lite6/visual/link3.obj"
         origin_xyz="0 0 0"
         origin_rpy="0 0 0" />
@@ -125,10 +125,10 @@
         origin_rpy="0 0 0"/>
       <xacro:common_link_visual
-        mesh_filename="lite6/visual/link4.stl"
-        origin_xyz="0 0 0"
-        origin_rpy="0 0 0"
-        material_name="${prefix}White" />
-      <xacro:common_link_collision
-        mesh_filename="lite6/visual/link4.stl"
+        mesh_filename="lite6/visual/link4.obj"
+        origin_xyz="0 0 0"
+        origin_rpy="0 0 0"
+        material_name="${prefix}White" />
+      <xacro:common_link_collision
+        mesh_filename="lite6/visual/link4.obj"
         origin_xyz="0 0 0"
         origin_rpy="0 0 0" />
@@ -151,10 +151,10 @@
         origin_rpy="0 0 0"/>
       <xacro:common_link_visual
-        mesh_filename="lite6/visual/link5.stl"
-        origin_xyz="0 0 0"
-        origin_rpy="0 0 0"
-        material_name="${prefix}White" />
-      <xacro:common_link_collision
-        mesh_filename="lite6/visual/link5.stl"
+        mesh_filename="lite6/visual/link5.obj"
+        origin_xyz="0 0 0"
+        origin_rpy="0 0 0"
+        material_name="${prefix}White" />
+      <xacro:common_link_collision
+        mesh_filename="lite6/visual/link5.obj"
         origin_xyz="0 0 0"
         origin_rpy="0 0 0" />
@@ -177,10 +177,10 @@
         origin_rpy="0 0 0"/>
       <xacro:common_link_visual
-        mesh_filename="lite6/visual/link6.stl"
+        mesh_filename="lite6/visual/link6.obj"
         origin_xyz="0 0 0"
         origin_rpy="0 0 0"
         material_name="${prefix}Silver" />
       <xacro:common_link_collision
-        mesh_filename="lite6/visual/link6.stl"
+        mesh_filename="lite6/visual/link6.obj"
         origin_xyz="0 0 0"
         origin_rpy="0 0 0" />

File: src/xarm_description/urdf/xarm_device_macro.xacro (robot description, xacro)
@@ -51,5 +51,8 @@
     </xacro:if>
     <xacro:unless value="${ros2_control_plugin == 'gazebo_ros2_control/GazeboSystem'}">
+      <!--
       <xacro:property name="mesh_path" value="package://xarm_description/meshes" scope="parent"/>
+      -->
+      <xacro:property name="mesh_path" value="$(arg xarm_description)/meshes" scope="parent"/>
     </xacro:unless>
     <!-- include common.link.xacro -->
