Commit message: trying out stuff

File: models/environment/lite6_table.urdf (robot description, URDF)
Before this commit: robot lite6_table, 3 links, 2 joints
Links:
- link link_lite6_table: mass None -> 10

File: models/objects/cube_1_inch.urdf (robot description, URDF)
Before this commit: robot cube_1_inch, 2 links, 0 joints
Links:
- link link_cube_1_inch: geometry collision box size=0.0244 0.0244 0.0244; collision sphere radius=1e-7
