Commit message: pick works!

File: models/objects/cube_1_inch_blue.urdf (robot description, URDF)
Before this commit: robot cube_1_inch, 2 links, 0 joints
Links:
- removed link link_cube_1_inch
- added link link_cube_1_inch_blue, mass 0.006; collision box size=0.0244 0.0244 0.0244; collision sphere radius=1e-7
